File: TasmoTree/TasmoTree.kicad_pcb (KiCad board)
At the start: 2 copper layers, 99.6 x 99.6 mm, 24 parts, among them J1 POWER_IN, J2 MOT_SW_CONN, J3 MOTOR_POWER, J4 LED_5MM_CONN, J5 LED_CONN_1, J6 LED_CONN_2, Q1 PSMN027-100PS, Q2 PSMN027-100PS, Q3 PSMN027-100PS, SW1 Rotary_Encoder_Switch, U1 ESP8266, U2 LD1117S33TR_SOT223, U3 LED-DRIVER, U4 LED-DRIVER, U5 LED-DRIVER

Commit message: generated gerber files and submitted for fabrication
Parts:
- added G***: LOGO, TasmoTree:TasmoTreeLogo, F.Cu at (126.0, 94.5)
- added G***: LOGO, TasmoTree:StanleySolutionsPCB_m, F.Cu at (102.6, 90.4)
-  : renamed from REF** (x4)
- moved   59.7 mm to (186.4, 142.7)
- moved   59.7 mm to (143.8, 64.0)
- moved   59.7 mm to (98.6, 76.2)
- moved   59.7 mm to (98.6, 108.7)
- moved C1 59.7 mm to (121.9, 62.5)
- moved C2 59.7 mm to (120.4, 55.4)
- moved Q3 59.7 mm to (159.5, 98.5)
- moved S1 59.7 mm to (149.4, 132.1)
- moved SW1 59.7 mm to (106.7, 133.6)
- moved U3 59.7 mm to (147.8, 86.4)
- moved U4 59.7 mm to (147.8, 71.6)
- moved U5 59.7 mm to (147.8, 56.4)
- moved J1 59.7 mm to (100.6, 67.6)
- moved J2 59.7 mm to (183.4, 119.5)
- moved J4 59.7 mm to (183.4, 101.1)
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Other:
- board text added: "12V+"
- board text added: "12V- (PWM)"
- board text added: "32V+"
- board text added: "GND"
- board text added: "NC"
- board text added: "RLY - NO"
- board text added: "TasmoTree For Shay"
- board text added: "V+"
- board text added: "V-"
- board text added: "©Stanley Solutions | 2020 Custom Crafted for Shay Hengen with love from Alan Hengen and Joe Stanley"
- board text added: "•"

Commit message: rev-2 design completed and ordered
Parts:
- U1: footprint TasmoTree:MODULE_ESP32-DEVKITC-32D -> TasmoTree:ESP8266_NODEMCU
- moved G*** 4.82 mm to (124.5, 89.9)
Connections:
- U1 pad 16: (no net) -> Net-(Q1-Pad1)
- U1 pad 17: (no net) -> Net-(Q2-Pad1)
- U1 pad 18: (no net) -> Net-(U1-Pad18)
- U1 pad 19: (no net) -> Net-(U1-Pad19)
- U1 pad 20: Net-(Q1-Pad1) -> Net-(U1-Pad20)
- U1 pad 21: Net-(Q2-Pad1) -> Net-(C2-Pad1)
- U1 pad 22: Net-(U1-Pad22) -> GNDPWR
- U1 pad 23: Net-(U1-Pad23) -> Net-(SW1-PadB)
- U1 pad 24: Net-(U1-Pad24) -> Net-(Q3-Pad1)
- U1 pad 25: Net-(C2-Pad1) -> Net-(R2-Pad2)
- U1 pad 26: GNDPWR -> Net-(R1-Pad2)
- U1 pad 27: Net-(SW1-PadB) -> Net-(U1-Pad27)
- U1 pad 28: Net-(Q3-Pad1) -> Net-(U1-Pad28)
- U1 pad 29: Net-(R2-Pad2) -> GNDPWR
- U1 pad 30: Net-(R1-Pad2) -> Net-(C2-Pad1)
- U3 pad 3: Net-(U1-Pad32) -> Net-(U1-Pad28)
- U3 pad 5: Net-(J6-Pad2) -> Net-(J6-Pad3)
- U3 pad 6: Net-(J6-Pad3) -> Net-(J6-Pad2)
- U4 pad 3: Net-(U1-Pad31) -> Net-(U1-Pad27)
- U4 pad 5: Net-(J5-Pad3) -> Net-(J6-Pad1)
- U4 pad 6: Net-(J6-Pad1) -> Net-(J5-Pad3)
- U5 pad 3: Net-(U1-Pad22) -> Net-(U1-Pad18)
- U5 pad 5: Net-(J5-Pad1) -> Net-(J5-Pad2)
- U5 pad 6: Net-(J5-Pad2) -> Net-(J5-Pad1)
Routing:
- net Net-(U1-Pad27): track 0.00 -> 37.8 mm
- net Net-(U1-Pad18): track 0.00 -> 36.7 mm
- net Net-(U1-Pad22): track 36.0 -> 0.00 mm
- net Net-(U1-Pad31): track 34.6 -> 0.00 mm
- net Net-(U1-Pad32): track 26.0 -> 0.00 mm
- net Net-(U1-Pad28): track 0.00 -> 26.0 mm
- net GNDPWR: track 278.8 -> 297.4 mm, vias 21 -> 13
- net Net-(J2-Pad2): track 86.8 -> 72.3 mm
- net Net-(Q2-Pad1): track 72.3 -> 86.8 mm
- net Net-(C2-Pad1): track 148.4 -> 159.6 mm
- net Net-(Q1-Pad2): track 37.3 -> 29.6 mm
- net Net-(J1-Pad4): track 89.9 -> 86.5 mm
- net Net-(Q1-Pad1): track 67.8 -> 71.0 mm
- net Net-(J3-Pad2): track 35.0 -> 37.8 mm
- net Net-(SW1-PadB): track 55.7 -> 53.2 mm
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Other:
- board text added: "MOTOR OUT"
