File: TasmoTree/TasmoTree.sch (KiCad schematic (older format))
At the start: 6 parts, among them Q1 PSMN027-100PS, U1 ESP32

Commit message: started pinout design and created symbol for led drivers
Parts:
- added J1: POWER_IN, symbol Connector:Screw_Terminal_01x04
- added J2: MOTOR_CONN, symbol Connector:Screw_Terminal_01x04
- added Q2: PSMN027-100PS, TO255P1040X460X2890-3, symbol TO220:STP24N60M6
- added U?: LED-DRIVER, symbol TasmoTree:LED-DRIVER
- gave numbers to parts that had none: 1
Connections:
- net labels added: 12V, 12VP, 32V
- wire segments 26 -> 48
Changed lines of the file:
@@
 $EndDescr
 $Comp
-L TO220:STP24N60M6 Q1
-U 1 1 5FC1E6D7
-P 6400 5000
-F 0 "Q1" H 6608 5046 50  0000 L CNN
-F 1 "PSMN027-100PS" H 6608 4955 50  0000 L CNN
-F 2 "TO255P1040X460X2890-3" H 6400 5000 50  0001 L BNN
-F 3 "" H 6400 5000 50  0001 L BNN
-F 4 "IPC-7251" H 6400 5000 50  0001 L BNN "STANDARD"
-F 5 "1" H 6400 5000 50  0001 L BNN "PARTREV"
-F 6 "STMicroelectronics" H 6400 5000 50  0001 L BNN "MANUFACTURER"
-	1    6400 5000
-	1    0    0    -1
-$EndComp
-$Comp
-L DPDTRelay:7-1393243-9 S1
-U 1 1 5FC1F173
-P 7800 3850
-F 0 "S1" H 7800 4617 50  0000 C CNN
-F 1 "EC2-12NU" H 7800 4526 50  0000 C CNN
-F 2 "RELAY_7-1393243-9" H 7800 3850 50  0001 L BNN
-F 3 "" H 7800 3850 50  0001 L BNN
-F 4 "7-1393243-9" H 7800 3850 50  0001 L BNN "Comment"
-	1    7800 3850
-	1    0    0    -1
-$EndComp
-$Comp
-L Regulator_Linear:LD1117S33TR_SOT223 U?
+L Regulator_Linear:LD1117S33TR_SOT223 U2
 U 1 1 5FC271A2
 P 1650 2800
-F 0 "U?" H 1650 3042 50  0000 C CNN
+F 0 "U2" H 1650 3042 50  0000 C CNN
 F 1 "LD1117S33TR_SOT223" H 1650 2951 50  0000 C CNN
 F 2 "Package_TO_SOT_SMD:SOT-223-3_TabPin2" H 1650 3000 50  0001 C CNN
@@
 	1    0    0    -1
 $EndComp
+Wire Wire Line
+	1950 2800 2050 2800
+Wire Wire Line
+	2050 2900 2050 2800
+Wire Wire Line
+	1150 2900 1150 2800
+Wire Wire Line
+	1150 2800 1350 2800
+Wire Wire Line
+	1150 3200 1650 3200
+Wire Wire Line
+	1650 3100 1650 3200
+Connection ~ 1650 3200
+Wire Wire Line
+	1650 3200 2050 3200
+Wire Wire Line
+	1650 3200 1650 5750
+Wire Wire Line
+	8000 4950 7550 4950
+Wire Wire Line
+	7550 5950 8000 5950
+Wire Wire Line
+	7700 5350 7550 5350
+Wire Wire Line
+	7700 5550 7700 5450
+Wire Wire Line
+	7550 5550 7700 5550
+Wire Wire Line
+	8150 5750 8150 6300
+Wire Wire Line
+	7550 5750 8150 5750
+Wire Wire Line
+	5850 5850 6750 5850
+$Comp
+L DPDTRelay:7-1393243-9 S1
+U 1 1 5FC1F173
+P 7150 5450
+F 0 "S1" H 7150 6217 50  0000 C CNN
+F 1 "EC2-12NU" H 7150 6126 50  0000 C CNN
+F 2 "RELAY_7-1393243-9" H 7150 5450 50  0001 L BNN
+F 3 "" H 7150 5450 50  0001 L BNN
+F 4 "7-1393243-9" H 7150 5450 50  0001 L BNN "Comment"
+	1    7150 5450
+	1    0    0    -1
+$EndComp
+$Comp
+L TO220:STP24N60M6 Q1
+U 1 1 5FC1E6D7
+P 5750 6600
+F 0 "Q1" H 5958 6646 50  0000 L CNN
+F 1 "PSMN027-100PS" H 5958 6555 50  0000 L CNN
+F 2 "TO255P1040X460X2890-3" H 5750 6600 50  0001 L BNN
+F 3 "" H 5750 6600 50  0001 L BNN
+F 4 "IPC-7251" H 5750 6600 50  0001 L BNN "STANDARD"
+F 5 "1" H 5750 6600 50  0001 L BNN "PARTREV"
+F 6 "STMicroelectronics" H 5750 6600 50  0001 L BNN "MANUFACTURER"
+	1    5750 6600
+	1    0    0    -1
+$EndComp
+Wire Wire Line
+	2700 4500 2500 4500
+Wire Wire Line
+	2700 2800 2050 2800
+Connection ~ 2050 2800
+Wire Wire Line
+	1650 5750 2500 5750
+Wire Wire Line
+	2500 5750 2500 4500
+Wire Wire Line
+	2500 5750 2500 7300
+Wire Wire Line
+	2500 7300 4500 7300
+Wire Wire Line
+	5850 7300 5850 6800
+Connection ~ 2500 5750
+$Comp
+L TasmoTree:LED-DRIVER U?
+U 1 1 5FC8124B
+P 7200 2700
+F 0 "U?" H 7200 2765 50  0000 C CNN
+F 1 "LED-DRIVER" H 7200 2674 50  0000 C CNN
+F 2 "" H 7150 2750 50  0001 C CNN
+F 3 "" H 7150 2750 50  0001 C CNN
+	1    7200 2700
+	1    0    0    -1
+$EndComp
+$Comp
+L TO220:STP24N60M6 Q2
+U 1 1 5FC8259F
+P 4400 6600
+F 0 "Q2" H 4608 6646 50  0000 L CNN
+F 1 "PSMN027-100PS" H 4608 6555 50  0000 L CNN
+F 2 "TO255P1040X460X2890-3" H 4400 6600 50  0001 L BNN
+F 3 "" H 4400 6600 50  0001 L BNN
+F 4 "IPC-7251" H 4400 6600 50  0001 L BNN "STANDARD"
+F 5 "1" H 4400 6600 50  0001 L BNN "PARTREV"
+F 6 "STMicroelectronics" H 4400 6600 50  0001 L BNN "MANUFACTURER"
+	1    4400 6600
+	1    0    0    -1
+$EndComp
+Wire Wire Line
+	4500 6800 4500 7300
+Connection ~ 4500 7300
+Wire Wire Line
+	4500 7300 5850 7300
+$Comp
+L Connector:Screw_Terminal_01x04 J1
+U 1 1 5FC98093
+P 1050 1750
+F 0 "J1" V 1014 1462 50  0000 R CNN
+F 1 "POWER_IN" V 923 1462 50  0000 R CNN
+F 2 "" H 1050 1750 50  0001 C CNN
+F 3 "~" H 1050 1750 50  0001 C CNN
+	1    1050 1750
+	0    -1   -1   0
+$EndComp
+Wire Wire Line
+	950  1950 950  2300
+Wire Wire Line
+	950  3200 1150 3200
+Connection ~ 1150 3200
+Wire Wire Line
+	1050 1950 1050 2800
+Wire Wire Line
+	1050 2800 1150 2800
+Connection ~ 1150 2800
+Wire Wire Line
+	1150 1950 1150 2300
+Wire Wire Line
+	1150 2300 950  2300
+Connection ~ 950  2300
+Wire Wire Line
+	950  2300 950  3200
+Text Label 950  1650 0    30   ~ 0
+12V
+Text Label 1150 1650 0    30   ~ 0
+32V
 $Comp
 L ESP32-DEVKITC-32D:ESP32-DEVKITC-32D U1
 U 1 1 5FC1B5D0
-P 4400 3700
-F 0 "U1" H 4400 4867 50  0000 C CNN
-F 1 "ESP32" H 4400 4776 50  0000 C CNN
-F 2 "MODULE_ESP32-DEVKITC-32D" H 4400 3700 50  0001 L BNN
-F 3 "" H 4400 3700 50  0001 L BNN
-F 4 "4" H 4400 3700 50  0001 L BNN "PARTREV"
-F 5 "Espressif Systems" H 4400 3700 50  0001 L BNN "MANUFACTURER"
-	1    4400 3700
-	1    0    0    -1
-$EndComp
-Wire Wire Line
-	1950 2800 2050 2800
-Wire Wire Line
-	2050 2900 2050 2800
-Connection ~ 2050 2800
-Wire Wire Line
-	2050 2800 3600 2800
-Wire Wire Line
-	1150 2900 1150 2800
-Wire Wire Line
-	1150 2800 1350 2800
-Wire Wire Line
-	1150 3200 1650 3200
-Wire Wire Line
-	1650 3100 1650 3200
-Connection ~ 1650 3200
-Wire Wire Line
-	1650 3200 2050 3200
-Wire Wire Line
-	6500 4800 6500 4700
-Wire Wire Line
-	6500 4250 7400 4250
-Wire Wire Line
-	8200 4150 8800 4150
-Wire Wire Line
-	8800 4150 8800 4700
-Wire Wire Line
-	8800 4700 6500 4700
-Connection ~ 6500 4700
-Wire Wire Line
-	6500 4700 6500 4250
-Wire Wire Line
-	8200 3950 8350 3950
-Wire Wire Line
-	8350 3950 8350 3750
-Wire Wire Line
-	8350 3750 8200 3750
-Wire Wire Line
-	8200 4350 8650 4350
-Wire Wire Line
-	8650 4350 8650 3350
-Wire Wire Line
-	8650 3350 8200 3350
-Wire Wire Line
-	1650 3200 1650 5750
-Wire Wire Line
-	1650 5750 3400 5750
-Wire Wire Line
-	6500 5750 6500 5200
-Wire Wire Line
-	3600 4500 3400 4500
-Wire Wire Line
-	3400 4500 3400 5750
-Connection ~ 3400 5750
-Wire Wire Line
-	3400 5750 6500 5750
+P 3500 3700
+F 0 "U1" H 3500 4867 50  0000 C CNN
+F 1 "ESP32" H 3500 4776 50  0000 C CNN
+F 2 "MODULE_ESP32-DEVKITC-32D" H 3500 3700 50  0001 L BNN
+F 3 "" H 3500 3700 50  0001 L BNN
+F 4 "4" H 3500 3700 50  0001 L BNN "PARTREV"
+F 5 "Espressif Systems" H 3500 3700 50  0001 L BNN "MANUFACTURER"
+	1    3500 3700
+	1    0    0    -1
+$EndComp
+Connection ~ 5850 6300
+Wire Wire Line
+	5850 6300 5850 5850
+Wire Wire Line
+	5850 6400 5850 6300
+Wire Wire Line
+	8150 6300 5850 6300
+$Comp
+L Connector:Screw_Terminal_01x04 J2
+U 1 1 5FC9C1FA
+P 8600 5250
+F 0 "J2" H 8680 5242 50  0000 L CNN
+F 1 "MOTOR_CONN" H 8680 5151 50  0000 L CNN
+F 2 "" H 8600 5250 50  0001 C CNN
+F 3 "~" H 8600 5250 50  0001 C CNN
+	1    8600 5250
+	1    0    0    -1
+$EndComp
+Text GLabel 1050 2450 2    50   Input ~ 0
+12VP
+Wire Wire Line
+	8400 5450 8100 5450
+Wire Wire Line
+	8400 5350 8000 5350
+Wire Wire Line
+	8400 5250 8100 5250
+Wire Wire Line
+	8100 4400 6500 4400
+Wire Wire Line
+	6500 4400 6500 5050
+Wire Wire Line
+	6500 5050 6750 5050
+Connection ~ 7700 5450
+Wire Wire Line
+	7700 5450 7700 5350
+Connection ~ 8000 5350
+Wire Wire Line
+	8000 5350 8000 5950
+Wire Wire Line
+	8000 4950 8000 5350
+Wire Wire Line
+	8100 4400 8100 5250
+Wire Wire Line
+	8400 5150 7550 5150
+Wire Wire Line
+	8100 5250 8100 5450
+Connection ~ 8100 5250
+Connection ~ 8100 5450
+Wire Wire Line
+	8100 5450 7700 5450
+Text GLabel 8250 5150 1    50   Input ~ 0
+12VP
 $EndSCHEMATC

Commit message: finished basic schematic layout
Parts:
- added J3: MOTOR_POWER, symbol Connector:Screw_Terminal_01x02
- added J4: LED_5MM_CONN, symbol Connector:Screw_Terminal_01x03
- added J5: LED_CONN_1, symbol Connector:Screw_Terminal_01x03
- added J6: LED_CONN_2, symbol Connector:Screw_Terminal_01x03
- added Q3: PSMN027-100PS, TO255P1040X460X2890-3, symbol TasmoTree-rescue:STP24N60M6-TO220
- added U2, U3: LED-DRIVER, symbol TasmoTree:LED-DRIVER
- J2: value MOTOR_CONN -> MOT_SW_CONN; symbol Connector:Screw_Terminal_01x04 -> Connector:Screw_Terminal_01x03
- Q1, Q2: symbol TO220:STP24N60M6 -> TasmoTree-rescue:STP24N60M6-TO220
- S1: symbol DPDTRelay:7-1393243-9 -> TasmoTree-rescue:7-1393243-9-DPDTRelay
- U1: value ESP32 -> ESP8266; symbol ESP32-DEVKITC-32D:ESP32-DEVKITC-32D -> TasmoTree-rescue:ESP8266-DEVKIT
- gave numbers to parts that had none: 1
Connections:
- net labels added: GNDPWR
- wire segments 48 -> 112
Other:
- moved on the sheet: U4

Commit message: resolved some issues with the ESP8266 symbol pinouts
Parts:
- renumbered U2 to U3, U3 to U4, U4 to U5
Connections:
- no-connect marks 0 -> 15
Changed lines of the file:
@@
 	1650 3200 2050 3200
-Wire Wire Line
-	1650 3200 1650 4300
 Wire Wire Line
 	8000 4950 7550 4950
@@
 	5850 7300 5850 6800
 $Comp
-L TasmoTree:LED-DRIVER U4
+L TasmoTree:LED-DRIVER U5
 U 1 1 5FC8124B
 P 5650 1650
-F 0 "U4" H 5650 1715 50  0000 C CNN
+F 0 "U5" H 5650 1715 50  0000 C CNN
 F 1 "LED-DRIVER" H 5650 1624 50  0000 C CNN
 F 2 "" H 5600 1700 50  0001 C CNN
@@
 	8000 5550 8000 5950
 $Comp
-L TasmoTree:LED-DRIVER U3
+L TasmoTree:LED-DRIVER U4
 U 1 1 5FC7CA67
 P 5650 2750
-F 0 "U3" H 5650 2815 50  0000 C CNN
+F 0 "U4" H 5650 2815 50  0000 C CNN
 F 1 "LED-DRIVER" H 5650 2724 50  0000 C CNN
 F 2 "" H 5600 2800 50  0001 C CNN
@@
 $EndComp
 $Comp
-L TasmoTree:LED-DRIVER U2
+L TasmoTree:LED-DRIVER U3
 U 1 1 5FC82B1A
 P 5650 3800
-F 0 "U2" H 5650 3865 50  0000 C CNN
+F 0 "U3" H 5650 3865 50  0000 C CNN
 F 1 "LED-DRIVER" H 5650 3774 50  0000 C CNN
 F 2 "" H 5600 3850 50  0001 C CNN
@@
 $EndComp
 $Comp
-L power:GNDPWR #PWR?
+L power:GNDPWR #PWR0101
 U 1 1 5FC83AC6
 P 950 3200
-F 0 "#PWR?" H 950 3000 50  0001 C CNN
+F 0 "#PWR0101" H 950 3000 50  0001 C CNN
 F 1 "GNDPWR" H 954 3046 50  0000 C CNN
 F 2 "" H 950 3150 50  0001 C CNN
@@
 Connection ~ 950  3200
 $Comp
-L power:GNDPWR #PWR?
+L power:GNDPWR #PWR0102
 U 1 1 5FC849DB
 P 5900 3500
-F 0 "#PWR?" H 5900 3300 50  0001 C CNN
+F 0 "#PWR0102" H 5900 3300 50  0001 C CNN
 F 1 "GNDPWR" H 5905 3345 50  0000 C CNN
 F 2 "" H 5900 3450 50  0001 C CNN
@@
 $EndComp
 $Comp
-L power:GNDPWR #PWR?
+L power:GNDPWR #PWR0103
 U 1 1 5FC85C75
 P 5900 2450
-F 0 "#PWR?" H 5900 2250 50  0001 C CNN
+F 0 "#PWR0103" H 5900 2250 50  0001 C CNN
 F 1 "GNDPWR" H 5905 2295 50  0000 C CNN
 F 2 "" H 5900 2400 50  0001 C CNN
@@
 $EndComp
 $Comp
-L power:GNDPWR #PWR?
+L power:GNDPWR #PWR0104
 U 1 1 5FC86A62
 P 5900 1350
-F 0 "#PWR?" H 5900 1150 50  0001 C CNN
+F 0 "#PWR0104" H 5900 1150 50  0001 C CNN
 F 1 "GNDPWR" H 5905 1195 50  0000 C CNN
 F 2 "" H 5900 1300 50  0001 C CNN
@@
 Wire Wire Line
 	4450 4300 2500 4300
-Connection ~ 1650 4300
 Wire Wire Line
 	1650 4300 1650 5750
@@
 Wire Wire Line
 	4750 2800 4750 1750
+Connection ~ 1650 4300
+Wire Wire Line
+	1650 3200 1650 4300
+NoConn ~ 2700 2300
+NoConn ~ 2700 2600
+NoConn ~ 2700 2700
+NoConn ~ 2700 2800
+NoConn ~ 2700 2900
+NoConn ~ 2700 3000
+NoConn ~ 2700 3100
+NoConn ~ 2700 3400
+NoConn ~ 2700 3500
+NoConn ~ 2700 3700
+NoConn ~ 4300 3300
+NoConn ~ 4300 3200
+NoConn ~ 4300 3000
+NoConn ~ 4300 2700
+NoConn ~ 4300 2600
 $EndSCHEMATC

Commit message: added missing rotary encoder
Parts:
- added R1, R2: R, symbol Device:R
- added SW1: Rotary_Encoder_Switch, symbol Device:Rotary_Encoder_Switch
Connections:
- net GNDPWR: now also SW1.C, SW1.S2
- net at C2.1, U1.11 (3v31), U1.21 (3v32)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: now also R1.1, R2.1
- net at U1.23 (GPIO14): now also R1.2, SW1.A
- net at U1.25 (GPIO13): now also SW1.S1
- net at U1.26 (GPIO15): now also R2.2, SW1.B
- no-connect marks 15 -> 12
Changed lines of the file:
@@
 Text Label 1150 1650 0    30   ~ 0
 32V
-$Comp
-L TasmoTree-rescue:ESP8266-DEVKIT U1
-U 1 1 5FC1B5D0
-P 3500 3200
-F 0 "U1" H 3500 4367 50  0000 C CNN
-F 1 "ESP8266" H 3500 4276 50  0000 C CNN
-F 2 "MODULE_ESP32-DEVKITC-32D" H 3500 3200 50  0001 L BNN
-F 3 "" H 3500 3200 50  0001 L BNN
-F 4 "4" H 3500 3200 50  0001 L BNN "PARTREV"
-F 5 "Espressif Systems" H 3500 3200 50  0001 L BNN "MANUFACTURER"
-	1    3500 3200
-	1    0    0    -1
-$EndComp
 Connection ~ 5850 6300
 Wire Wire Line
@@
 	3350 7300 4500 7300
 Wire Wire Line
-	4300 2400 4950 2400
-Wire Wire Line
-	4950 2400 4950 5950
-Wire Wire Line
-	4950 5950 4300 5950
+	5250 2400 5250 5950
 Wire Wire Line
 	4300 5950 4300 6700
@@
 	1    0    0    -1
 $EndComp
-Text GLabel 3800 5250 1    50   Input ~ 0
+Text GLabel 3800 5300 1    50   Input ~ 0
 12VP
-Wire Wire Line
-	3800 5450 3800 5250
 Wire Wire Line
 	3800 5550 3350 5550
@@
 	7050 1350 7050 2550
 Wire Wire Line
-	4300 3700 4750 3700
+	4300 3700 4700 3700
 Wire Wire Line
 	4750 3700 4750 2800
@@
 NoConn ~ 2700 3500
 NoConn ~ 2700 3700
-NoConn ~ 4300 3300
-NoConn ~ 4300 3200
-NoConn ~ 4300 3000
 NoConn ~ 4300 2700
 NoConn ~ 4300 2600
+$Comp
+L Device:Rotary_Encoder_Switch SW1
+U 1 1 5FD20C7F
+P 4600 5000
+F 0 "SW1" H 4600 5367 50  0000 C CNN
+F 1 "Rotary_Encoder_Switch" H 4600 5276 50  0000 C CNN
+F 2 "" H 4450 5160 50  0001 C CNN
+F 3 "~" H 4600 5260 50  0001 C CNN
+	1    4600 5000
+	1    0    0    -1
+$EndComp
+Wire Wire Line
+	4300 5950 5250 5950
+Wire Wire Line
+	4300 2400 5250 2400
+Wire Wire Line
+	5200 4900 5200 3200
+$Comp
+L TasmoTree-rescue:ESP8266-DEVKIT U1
+U 1 1 5FC1B5D0
+P 3500 3200
+F 0 "U1" H 3500 4367 50  0000 C CNN
+F 1 "ESP8266" H 3500 4276 50  0000 C CNN
+F 2 "MODULE_ESP32-DEVKITC-32D" H 3500 3200 50  0001 L BNN
+F 3 "" H 3500 3200 50  0001 L BNN
+F 4 "4" H 3500 3200 50  0001 L BNN "PARTREV"
+F 5 "Espressif Systems" H 3500 3200 50  0001 L BNN "MANUFACTURER"
+	1    3500 3200
+	1    0    0    -1
+$EndComp
+Wire Wire Line
+	4300 3000 4550 3000
+Wire Wire Line
+	4550 4400 4050 4400
+Wire Wire Line
+	4050 4400 4050 4900
+Wire Wire Line
+	4050 4900 4300 4900
+Wire Wire Line
+	4300 5100 4100 5100
+Wire Wire Line
+	4100 5100 4100 4450
+Wire Wire Line
+	4100 4450 4600 4450
+Wire Wire Line
+	4600 4450 4600 3300
+Wire Wire Line
+	4600 3300 4300 3300
+Wire Wire Line
+	4300 5000 4000 5000
+Wire Wire Line
+	2500 5000 2500 5750
+Connection ~ 2500 5750
+Wire Wire Line
+	4000 5000 4000 5300
+Wire Wire Line
+	4000 5300 4900 5300
+Wire Wire Line
+	4900 5300 4900 5100
+Connection ~ 4000 5000
+Wire Wire Line
+	4000 5000 2500 5000
+Wire Wire Line
+	3800 5450 3800 5300
+$Comp
+L Device:R R1
+U 1 1 5FD60931
+P 4700 4150
+F 0 "R1" H 4770 4196 50  0000 L CNN
+F 1 "R" H 4770 4105 50  0000 L CNN
+F 2 "" V 4630 4150 50  0001 C CNN
+F 3 "~" H 4700 4150 50  0001 C CNN
+	1    4700 4150
+	1    0    0    -1
+$EndComp
+$Comp
+L Device:R R2
+U 1 1 5FD612A1
+P 4950 4150
+F 0 "R2" H 5020 4196 50  0000 L CNN
+F 1 "R" H 5020 4105 50  0000 L CNN
+F 2 "" V 4880 4150 50  0001 C CNN
+F 3 "~" H 4950 4150 50  0001 C CNN
+	1    4950 4150
+	1    0    0    -1
+$EndComp
+Wire Wire Line
+	4700 4000 4700 3700
+Connection ~ 4700 3700
+Wire Wire Line
+	4700 3700 4750 3700
+Wire Wire Line
+	4750 3700 4950 3700
+Wire Wire Line
+	4950 3700 4950 4000
+Connection ~ 4750 3700
+Wire Wire Line
+	4950 4300 4950 4450
+Wire Wire Line
+	4950 4450 4600 4450
+Connection ~ 4600 4450
+Wire Wire Line
+	4550 4400 4700 4400
+Wire Wire Line
+	4700 4400 4700 4300
+Connection ~ 4550 4400
+Wire Wire Line
+	4550 3000 4550 4400
+Wire Wire Line
+	4900 4900 5200 4900
+Wire Wire Line
+	4300 3200 5200 3200
 $EndSCHEMATC
